File: Hardware/nucular-keyboard.sch (KiCad schematic (older format))
At the start: 34 parts, among them IC1 STM32L052R6Tx, J1 JAE_AA01B-S040VA1, J2 JAE_KX14-40K2D, J3 CONN_01X16, J4 CONN_01X03, Q1 IRLML6402, U1 MCP1700T-3302E/MB

Commit message: Updated all footprints
Parts:
- C1, C2, C5, C6, C7, C8, C9: footprint Capacitors_SMD:C_0402 -> Capacitor_SMD:C_0402_1005Metric; symbol C -> nucular-keyboard-rescue:C
- C3, C4: footprint Capacitors_SMD:C_0603 -> Capacitor_SMD:C_0603_1608Metric; symbol C -> nucular-keyboard-rescue:C
- D1: symbol Nexperia_PRTR5V0U2X -> 000-Components:Nexperia_PRTR5V0U2X
- IC1: symbol STM32L052R6Tx -> nucular-keyboard-rescue:STM32L052R6Tx
- J1: symbol JAE_AA01B-S040VA1 -> 000-Components:JAE_AA01B-S040VA1
- J2: symbol JAE_KX14-40K2D -> 000-Components:JAE_KX14-40K2D
- J3: symbol CONN_01X16 -> nucular-keyboard-rescue:CONN_01X16
- J4: symbol CONN_01X03 -> nucular-keyboard-rescue:CONN_01X03
- JPA4, JPA5, JPC4, JPC5: symbol TEST_1P -> nucular-keyboard-rescue:TEST_1P
- Q1: symbol BSS84 -> nucular-keyboard-rescue:BSS84
- R1, R10, R11, R12, R2, R3, R4, R5, R6, R7, R8, R9: footprint Resistors_SMD:R_0402 -> Resistor_SMD:R_0402_1005Metric; symbol R -> nucular-keyboard-rescue:R
- U1: footprint 000-Modules:SOT89-3 -> Package_TO_SOT_SMD:SOT-89-3; symbol Microchip_MCP1700T-3302E/MB -> nucular-keyboard-rescue:Microchip_MCP1700T-3302E_MB
- USB1: symbol USB_OTG -> nucular-keyboard-rescue:USB_OTG

Commit message: Saved same to schematic
Parts:
- D1: footprint 000-Modules:SOT143B -> Package_TO_SOT_SMD:SOT-143
- IC1: footprint Housings_QFP:LQFP-64_10x10mm_Pitch0.5mm -> Package_QFP:LQFP-64_10x10mm_P0.5mm
- J3: footprint Pin_Headers:Pin_Header_Straight_1x16_Pitch2.54mm -> Connector_PinHeader_2.54mm:PinHeader_1x16_P2.54mm_Vertical
- J4: footprint Pin_Headers:Pin_Header_Straight_1x03_Pitch2.54mm -> Connector_PinHeader_2.54mm:PinHeader_1x03_P2.54mm_Vertical
- JPA4, JPA5, JPC4, JPC5: footprint Wire_Pads:SolderWirePad_single_0-8mmDrill -> TestPoint:TestPoint_THTPad_D1.0mm_Drill0.5mm
- Q1: footprint TO_SOT_Packages_SMD:SOT-23 -> Package_TO_SOT_SMD:SOT-23
Changed lines of the file:
@@
 F 0 "J3" H 10850 5400 50  0000 L CNN
 F 1 "CONN_01X16" H 11000 5400 50  0000 L CNN
-F 2 "Pin_Headers:Pin_Header_Straight_1x16_Pitch2.54mm" H 11450 6250 50  0001 C CNN
+F 2 "Connector_PinHeader_2.54mm:PinHeader_1x16_P2.54mm_Vertical" H 11450 6250 50  0001 C CNN
 F 3 "" H 11450 6250 50  0001 C CNN
 	1    11450 6250
@@
 F 0 "J4" H 10850 7550 50  0000 L CNN
 F 1 "CONN_01X03" H 11000 7550 50  0000 L CNN
-F 2 "Pin_Headers:Pin_Header_Straight_1x03_Pitch2.54mm" H 11450 7750 50  0001 C CNN
+F 2 "Connector_PinHeader_2.54mm:PinHeader_1x03_P2.54mm_Vertical" H 11450 7750 50  0001 C CNN
 F 3 "" H 11450 7750 50  0001 C CNN
 	1    11450 7750
@@
 F 0 "JPC4" V 1700 4550 50  0000 C CNN
 F 1 "TEST_1P" V 1700 4600 50  0001 C CNN
-F 2 "Wire_Pads:SolderWirePad_single_0-8mmDrill" H 1900 4250 50  0001 C CNN
+F 2 "TestPoint:TestPoint_THTPad_D1.0mm_Drill0.5mm" H 1900 4250 50  0001 C CNN
 F 3 "" H 1900 4250 50  0001 C CNN
 	1    1700 4250
@@
 F 0 "JPC5" V 1700 4650 50  0000 C CNN
 F 1 "TEST_1P" V 1700 4700 50  0001 C CNN
-F 2 "Wire_Pads:SolderWirePad_single_0-8mmDrill" H 1900 4350 50  0001 C CNN
+F 2 "TestPoint:TestPoint_THTPad_D1.0mm_Drill0.5mm" H 1900 4350 50  0001 C CNN
 F 3 "" H 1900 4350 50  0001 C CNN
 	1    1700 4350
@@
 F 0 "JPA4" V 9000 2850 50  0000 C CNN
 F 1 "TEST_1P" V 9000 2900 50  0001 C CNN
-F 2 "Wire_Pads:SolderWirePad_single_0-8mmDrill" H 9200 2550 50  0001 C CNN
+F 2 "TestPoint:TestPoint_THTPad_D1.0mm_Drill0.5mm" H 9200 2550 50  0001 C CNN
 F 3 "" H 9200 2550 50  0001 C CNN
 	1    9000 2550
@@
 F 0 "JPA5" V 9000 2950 50  0000 C CNN
 F 1 "TEST_1P" V 9000 3000 50  0001 C CNN
-F 2 "Wire_Pads:SolderWirePad_single_0-8mmDrill" H 9200 2650 50  0001 C CNN
+F 2 "TestPoint:TestPoint_THTPad_D1.0mm_Drill0.5mm" H 9200 2650 50  0001 C CNN
 F 3 "" H 9200 2650 50  0001 C CNN
 	1    9000 2650
@@
 F 0 "IC1" H 2750 5850 50  0000 C CNN
 F 1 "STM32L052R6Tx" H 2750 5750 50  0000 C CNN
-F 2 "Housings_QFP:LQFP-64_10x10mm_Pitch0.5mm" H 8250 5625 50  0001 R TNN
+F 2 "Package_QFP:LQFP-64_10x10mm_P0.5mm" H 8250 5625 50  0001 R TNN
 F 3 "" H 5350 3650 50  0001 C CNN
 	1    5350 3650
@@
 F 0 "Q1" V 7343 7600 50  0000 C CNN
 F 1 "IRLML6402" V 7252 7600 50  0000 C CNN
-F 2 "TO_SOT_Packages_SMD:SOT-23" H 7200 7525 50  0001 L CIN
+F 2 "Package_TO_SOT_SMD:SOT-23" H 7200 7525 50  0001 L CIN
 F 3 "" H 7000 7600 50  0001 L CNN
 	1    7000 7600
@@
 F 0 "D1" H 3800 7863 60  0000 C CNN
 F 1 "PRTR5V0U2X" H 3800 7969 60  0000 C CNN
-F 2 "000-Modules:SOT143B" H 3700 8600 60  0001 C CNN
+F 2 "Package_TO_SOT_SMD:SOT-143" H 3700 8600 60  0001 C CNN
 F 3 "" H 3700 8600 60  0001 C CNN
 	1    3800 8350

Commit message: Finished routing
Parts:
- C1, C2, C5, C6, C7, C8, C9: footprint Capacitor_SMD:C_0402_1005Metric -> Capacitor_SMD:C_0603_1608Metric
- R1, R10, R11, R12, R2, R3, R4, R5, R6, R7, R8, R9: footprint Resistor_SMD:R_0402_1005Metric -> Resistor_SMD:R_0603_1608Metric
Changed lines of the file:
@@
 F 0 "C6" H 6315 9646 50  0000 L CNN
 F 1 "100n" H 6315 9555 50  0000 L CNN
-F 2 "Capacitor_SMD:C_0402_1005Metric" H 6238 9450 50  0001 C CNN
+F 2 "Capacitor_SMD:C_0603_1608Metric" H 6238 9450 50  0001 C CNN
 F 3 "" H 6200 9600 50  0001 C CNN
 	1    6200 9600
@@
 F 0 "C1" H 1565 2596 50  0000 L CNN
 F 1 "100n" H 1565 2505 50  0000 L CNN
-F 2 "Capacitor_SMD:C_0402_1005Metric" H 1488 2400 50  0001 C CNN
+F 2 "Capacitor_SMD:C_0603_1608Metric" H 1488 2400 50  0001 C CNN
 F 3 "" H 1450 2550 50  0001 C CNN
 	1    1450 2550
@@
 F 0 "R1" V 13900 6150 50  0000 C CNN
 F 1 "100R" V 13900 5650 50  0000 C CNN
-F 2 "Resistor_SMD:R_0402_1005Metric" V 13780 5900 50  0001 C CNN
+F 2 "Resistor_SMD:R_0603_1608Metric" V 13780 5900 50  0001 C CNN
 F 3 "" H 13850 5900 50  0001 C CNN
 	1    13850 5900
@@
 F 0 "R2" V 13900 6250 50  0000 C CNN
 F 1 "100R" V 13900 5750 50  0000 C CNN
-F 2 "Resistor_SMD:R_0402_1005Metric" V 13780 6000 50  0001 C CNN
+F 2 "Resistor_SMD:R_0603_1608Metric" V 13780 6000 50  0001 C CNN
 F 3 "" H 13850 6000 50  0001 C CNN
 	1    13850 6000
@@
 F 0 "R3" V 13900 6350 50  0000 C CNN
 F 1 "100R" V 13900 5850 50  0000 C CNN
-F 2 "Resistor_SMD:R_0402_1005Metric" V 13780 6100 50  0001 C CNN
+F 2 "Resistor_SMD:R_0603_1608Metric" V 13780 6100 50  0001 C CNN
 F 3 "" H 13850 6100 50  0001 C CNN
 	1    13850 6100
@@
 F 0 "R4" V 13900 6450 50  0000 C CNN
 F 1 "100R" V 13900 5950 50  0000 C CNN
-F 2 "Resistor_SMD:R_0402_1005Metric" V 13780 6200 50  0001 C CNN
+F 2 "Resistor_SMD:R_0603_1608Metric" V 13780 6200 50  0001 C CNN
 F 3 "" H 13850 6200 50  0001 C CNN
 	1    13850 6200
@@
 F 0 "R5" H 14020 7396 50  0000 L CNN
 F 1 "4k7" H 14020 7305 50  0000 L CNN
-F 2 "Resistor_SMD:R_0402_1005Metric" V 13880 7350 50  0001 C CNN
+F 2 "Resistor_SMD:R_0603_1608Metric" V 13880 7350 50  0001 C CNN
 F 3 "" H 13950 7350 50  0001 C CNN
 	1    13950 7350
@@
 F 0 "R6" H 14470 7396 50  0000 L CNN
 F 1 "4k7" H 14470 7305 50  0000 L CNN
-F 2 "Resistor_SMD:R_0402_1005Metric" V 14330 7350 50  0001 C CNN
+F 2 "Resistor_SMD:R_0603_1608Metric" V 14330 7350 50  0001 C CNN
 F 3 "" H 14400 7350 50  0001 C CNN
 	1    14400 7350
@@
 F 0 "R7" H 14870 7396 50  0000 L CNN
 F 1 "4k7" H 14870 7305 50  0000 L CNN
-F 2 "Resistor_SMD:R_0402_1005Metric" V 14730 7350 50  0001 C CNN
+F 2 "Resistor_SMD:R_0603_1608Metric" V 14730 7350 50  0001 C CNN
 F 3 "" H 14800 7350 50  0001 C CNN
 	1    14800 7350
@@
 F 0 "R8" H 6470 7896 50  0000 L CNN
 F 1 "4k7" H 6470 7805 50  0000 L CNN
-F 2 "Resistor_SMD:R_0402_1005Metric" V 6330 7850 50  0001 C CNN
+F 2 "Resistor_SMD:R_0603_1608Metric" V 6330 7850 50  0001 C CNN
 F 3 "" H 6400 7850 50  0001 C CNN
 	1    6400 7850
@@
 F 0 "C2" H 7665 7896 50  0000 L CNN
 F 1 "100n" H 7665 7805 50  0000 L CNN
-F 2 "Capacitor_SMD:C_0402_1005Metric" H 7588 7700 50  0001 C CNN
+F 2 "Capacitor_SMD:C_0603_1608Metric" H 7588 7700 50  0001 C CNN
 F 3 "" H 7550 7850 50  0001 C CNN
 	1    7550 7850
@@
 F 0 "C5" H 5865 9646 50  0000 L CNN
 F 1 "100n" H 5865 9555 50  0000 L CNN
-F 2 "Capacitor_SMD:C_0402_1005Metric" H 5788 9450 50  0001 C CNN
+F 2 "Capacitor_SMD:C_0603_1608Metric" H 5788 9450 50  0001 C CNN
 F 3 "" H 5750 9600 50  0001 C CNN
 	1    5750 9600
@@
 F 0 "C9" H 7665 9646 50  0000 L CNN
 F 1 "100n" H 7665 9555 50  0000 L CNN
-F 2 "Capacitor_SMD:C_0402_1005Metric" H 7588 9450 50  0001 C CNN
+F 2 "Capacitor_SMD:C_0603_1608Metric" H 7588 9450 50  0001 C CNN
 F 3 "" H 7550 9600 50  0001 C CNN
 	1    7550 9600
@@
 F 0 "C8" H 7215 9646 50  0000 L CNN
 F 1 "100n" H 7215 9555 50  0000 L CNN
-F 2 "Capacitor_SMD:C_0402_1005Metric" H 7138 9450 50  0001 C CNN
+F 2 "Capacitor_SMD:C_0603_1608Metric" H 7138 9450 50  0001 C CNN
 F 3 "" H 7100 9600 50  0001 C CNN
 	1    7100 9600
@@
 F 0 "C7" H 6765 9646 50  0000 L CNN
 F 1 "100n" H 6765 9555 50  0000 L CNN
-F 2 "Capacitor_SMD:C_0402_1005Metric" H 6688 9450 50  0001 C CNN
+F 2 "Capacitor_SMD:C_0603_1608Metric" H 6688 9450 50  0001 C CNN
 F 3 "" H 6650 9600 50  0001 C CNN
 	1    6650 9600
@@
 F 0 "R12" V 13900 5750 50  0000 C CNN
 F 1 "100R" V 13900 5250 50  0000 C CNN
-F 2 "Resistor_SMD:R_0402_1005Metric" V 13780 5500 50  0001 C CNN
+F 2 "Resistor_SMD:R_0603_1608Metric" V 13780 5500 50  0001 C CNN
 F 3 "" H 13850 5500 50  0001 C CNN
 	1    13850 5500
@@
 F 0 "R9" V 13900 5850 50  0000 C CNN
 F 1 "100R" V 13900 5350 50  0000 C CNN
-F 2 "Resistor_SMD:R_0402_1005Metric" V 13780 5600 50  0001 C CNN
+F 2 "Resistor_SMD:R_0603_1608Metric" V 13780 5600 50  0001 C CNN
 F 3 "" H 13850 5600 50  0001 C CNN
 	1    13850 5600
@@
 F 0 "R10" V 13900 5950 50  0000 C CNN
 F 1 "100R" V 13900 5450 50  0000 C CNN
-F 2 "Resistor_SMD:R_0402_1005Metric" V 13780 5700 50  0001 C CNN
+F 2 "Resistor_SMD:R_0603_1608Metric" V 13780 5700 50  0001 C CNN
 F 3 "" H 13850 5700 50  0001 C CNN
 	1    13850 5700
@@
 F 0 "R11" V 13900 6050 50  0000 C CNN
 F 1 "100R" V 13900 5550 50  0000 C CNN
-F 2 "Resistor_SMD:R_0402_1005Metric" V 13780 5800 50  0001 C CNN
+F 2 "Resistor_SMD:R_0603_1608Metric" V 13780 5800 50  0001 C CNN
 F 3 "" H 13850 5800 50  0001 C CNN
 	1    13850 5800

Commit message: Add silkscreen to back side
Parts:
- C1, C2, C5, C6, C7, C8, C9: JLC_Part. No. (none) -> C143640
- C3, C4: JLC_Part. No. (none) -> C162270
- D1: JLC_Part. No. (none) -> C12333
- IC1: JLC_Part. No. (none) -> C139720
- Q1: JLC_Part. No. (none) -> C2593
- R1, R10, R11, R12, R2, R3, R4, R9: JLC_Part. No. (none) -> C441916
- R5, R6, R7, R8: JLC_Part. No. (none) -> C278604
- U1: JLC_Part. No. (none) -> C39051
Changed lines of the file:
@@
 F 2 "Capacitor_SMD:C_0603_1608Metric" H 6238 9450 50  0001 C CNN
 F 3 "" H 6200 9600 50  0001 C CNN
+F 4 "C143640" H 6200 9600 50  0001 C CNN "JLC_Part. No."
 	1    6200 9600
 	1    0    0    -1
@@
 F 2 "Capacitor_SMD:C_0603_1608Metric" H 1488 2400 50  0001 C CNN
 F 3 "" H 1450 2550 50  0001 C CNN
+F 4 "C143640" H 1450 2550 50  0001 C CNN "JLC_Part. No."
 	1    1450 2550
 	-1   0    0    -1
@@
 F 2 "Resistor_SMD:R_0603_1608Metric" V 13780 5900 50  0001 C CNN
 F 3 "" H 13850 5900 50  0001 C CNN
+F 4 "C441916" H 13850 5900 50  0001 C CNN "JLC_Part. No."
 	1    13850 5900
 	0    -1   -1   0
@@
 F 2 "Resistor_SMD:R_0603_1608Metric" V 13780 6000 50  0001 C CNN
 F 3 "" H 13850 6000 50  0001 C CNN
+F 4 "C441916" H 13850 6000 50  0001 C CNN "JLC_Part. No."
 	1    13850 6000
 	0    -1   -1   0
@@
 F 2 "Resistor_SMD:R_0603_1608Metric" V 13780 6100 50  0001 C CNN
 F 3 "" H 13850 6100 50  0001 C CNN
+F 4 "C441916" H 13850 6100 50  0001 C CNN "JLC_Part. No."
 	1    13850 6100
 	0    -1   -1   0
@@
 F 2 "Resistor_SMD:R_0603_1608Metric" V 13780 6200 50  0001 C CNN
 F 3 "" H 13850 6200 50  0001 C CNN
+F 4 "C441916" H 13850 6200 50  0001 C CNN "JLC_Part. No."
 	1    13850 6200
 	0    -1   -1   0
@@
 F 2 "Resistor_SMD:R_0603_1608Metric" V 13880 7350 50  0001 C CNN
 F 3 "" H 13950 7350 50  0001 C CNN
+F 4 "C278604" H 13950 7350 50  0001 C CNN "JLC_Part. No."
 	1    13950 7350
 	1    0    0    -1
@@
 F 2 "Resistor_SMD:R_0603_1608Metric" V 14330 7350 50  0001 C CNN
 F 3 "" H 14400 7350 50  0001 C CNN
+F 4 "C278604" H 14400 7350 50  0001 C CNN "JLC_Part. No."
 	1    14400 7350
 	1    0    0    -1
@@
 F 2 "Resistor_SMD:R_0603_1608Metric" V 14730 7350 50  0001 C CNN
 F 3 "" H 14800 7350 50  0001 C CNN
+F 4 "C278604" H 14800 7350 50  0001 C CNN "JLC_Part. No."
 	1    14800 7350
 	1    0    0    -1
@@
 F 2 "Resistor_SMD:R_0603_1608Metric" V 6330 7850 50  0001 C CNN
 F 3 "" H 6400 7850 50  0001 C CNN
+F 4 "C278604" H 6400 7850 50  0001 C CNN "JLC_Part. No."
 	1    6400 7850
 	1    0    0    -1
@@
 F 2 "Capacitor_SMD:C_0603_1608Metric" H 7588 7700 50  0001 C CNN
 F 3 "" H 7550 7850 50  0001 C CNN
+F 4 "C143640" H 7550 7850 50  0001 C CNN "JLC_Part. No."
 	1    7550 7850
 	1    0    0    -1
@@
 F 2 "Capacitor_SMD:C_0603_1608Metric" H 2888 9550 50  0001 C CNN
 F 3 "" H 2850 9700 50  0001 C CNN
+F 4 "C162270" H 2850 9700 50  0001 C CNN "JLC_Part. No."
 	1    2850 9700
 	1    0    0    -1
@@
 F 2 "Capacitor_SMD:C_0603_1608Metric" H 4588 9550 50  0001 C CNN
 F 3 "" H 4550 9700 50  0001 C CNN
+F 4 "C162270" H 4550 9700 50  0001 C CNN "JLC_Part. No."
 	1    4550 9700
 	1    0    0    -1
@@
 F 2 "Capacitor_SMD:C_0603_1608Metric" H 5788 9450 50  0001 C CNN
 F 3 "" H 5750 9600 50  0001 C CNN
+F 4 "C143640" H 5750 9600 50  0001 C CNN "JLC_Part. No."
 	1    5750 9600
 	1    0    0    -1
@@
 F 2 "Capacitor_SMD:C_0603_1608Metric" H 7588 9450 50  0001 C CNN
 F 3 "" H 7550 9600 50  0001 C CNN
+F 4 "C143640" H 7550 9600 50  0001 C CNN "JLC_Part. No."
 	1    7550 9600
 	1    0    0    -1
@@
 F 2 "Capacitor_SMD:C_0603_1608Metric" H 7138 9450 50  0001 C CNN
 F 3 "" H 7100 9600 50  0001 C CNN
+F 4 "C143640" H 7100 9600 50  0001 C CNN "JLC_Part. No."
 	1    7100 9600
 	1    0    0    -1
@@
 F 2 "Capacitor_SMD:C_0603_1608Metric" H 6688 9450 50  0001 C CNN
 F 3 "" H 6650 9600 50  0001 C CNN
+F 4 "C143640" H 6650 9600 50  0001 C CNN "JLC_Part. No."
 	1    6650 9600
 	1    0    0    -1
@@
 F 2 "Resistor_SMD:R_0603_1608Metric" V 13780 5500 50  0001 C CNN
 F 3 "" H 13850 5500 50  0001 C CNN
+F 4 "C441916" H 13850 5500 50  0001 C CNN "JLC_Part. No."
 	1    13850 5500
 	0    -1   -1   0
@@
 F 2 "Resistor_SMD:R_0603_1608Metric" V 13780 5600 50  0001 C CNN
 F 3 "" H 13850 5600 50  0001 C CNN
+F 4 "C441916" H 13850 5600 50  0001 C CNN "JLC_Part. No."
 	1    13850 5600
 	0    -1   -1   0
@@
 F 2 "Resistor_SMD:R_0603_1608Metric" V 13780 5700 50  0001 C CNN
 F 3 "" H 13850 5700 50  0001 C CNN
+F 4 "C441916" H 13850 5700 50  0001 C CNN "JLC_Part. No."
 	1    13850 5700
 	0    -1   -1   0
@@
 F 2 "Resistor_SMD:R_0603_1608Metric" V 13780 5800 50  0001 C CNN
 F 3 "" H 13850 5800 50  0001 C CNN
+F 4 "C441916" H 13850 5800 50  0001 C CNN "JLC_Part. No."
 	1    13850 5800
 	0    -1   -1   0
@@
 F 2 "Package_QFP:LQFP-64_10x10mm_P0.5mm" H 8250 5625 50  0001 R TNN
 F 3 "" H 5350 3650 50  0001 C CNN
+F 4 "C139720" H 5350 3650 50  0001 C CNN "JLC_Part. No."
 	1    5350 3650
 	1    0    0    -1
@@
 F 2 "Package_TO_SOT_SMD:SOT-23" H 7200 7525 50  0001 L CIN
 F 3 "" H 7000 7600 50  0001 L CNN
+F 4 "C2593" H 7000 7600 50  0001 C CNN "JLC_Part. No."
 	1    7000 7600
 	0    1    -1   0
@@
 F 2 "Package_TO_SOT_SMD:SOT-143" H 3700 8600 60  0001 C CNN
 F 3 "" H 3700 8600 60  0001 C CNN
+F 4 "C12333" H 3800 8350 50  0001 C CNN "JLC_Part. No."
 	1    3800 8350
 	-1   0    0    1
@@
 F 2 "Package_TO_SOT_SMD:SOT-89-3" H 3800 9050 50  0001 C CNN
 F 3 "" H 3800 9500 50  0001 C CNN
+F 4 "C39051" H 3800 9400 50  0001 C CNN "JLC_Part. No."
 	1    3800 9400
 	1    0    0    -1
